File: Board_Design/WS2812_Driver.sch (KiCad schematic (older format))
At the start: 22 parts, among them J1 5Vin, J10 PogoPin, J11 PogoPin, J12 PogoPin, J2 GNDin, J3 5Vout, J4 DOUT, J5 GNDout, J6 INPUT, J7 PogoPin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

Commit message: Updated for DFR
Updated design for more design-for-manufacturability.
Connections:
- net GND: now also J6.7 (Pin_7); no longer J6.8 (Pin_8)
- net SPI_MOSI: now also J6.8 (Pin_8); no longer J6.7 (Pin_7)
Changed lines of the file:
@@
 	1    0    0    -1
 $EndComp
-Text GLabel 6850 5600 0    50   Input ~ 0
+Text GLabel 7650 5600 2    50   Input ~ 0
 SPI_MOSI
 Wire Wire Line
@@
 SPI_MISO
 Wire Wire Line
-	6850 5600 7000 5600
+	7650 5600 7500 5600
 $Comp
 L power:+3.3V #PWR0117
@@
 L power:GND #PWR0118
 U 1 1 61B38A83
-P 7750 5825
-F 0 "#PWR0118" H 7750 5575 50  0001 C CNN
-F 1 "GND" H 7755 5652 50  0000 C CNN
-F 2 "" H 7750 5825 50  0001 C CNN
-F 3 "" H 7750 5825 50  0001 C CNN
-	1    7750 5825
-	1    0    0    -1
+P 6750 5825
+F 0 "#PWR0118" H 6750 5575 50  0001 C CNN
+F 1 "GND" H 6755 5652 50  0000 C CNN
+F 2 "" H 6750 5825 50  0001 C CNN
+F 3 "" H 6750 5825 50  0001 C CNN
+	1    6750 5825
+	-1   0    0    -1
 $EndComp
 Wire Wire Line
-	7750 5825 7750 5600
+	6750 5825 6750 5600
 Wire Wire Line
-	7750 5600 7500 5600
+	6750 5600 7000 5600
 NoConn ~ 7500 5300
 $Comp
